File: BoxPad_PCB/BoxPad_PCB.kicad_sch (KiCad schematic)
At the start: 20 parts, among them SW1 SW_Push_45deg, SW2 SW_Push_45deg, SW3 SW_Push_45deg, SW4 SW_Push_45deg, SW5 SW_Push_45deg, SW6 SW_Push_45deg, SW7 SW_Push_45deg, SW8 SW_Push_45deg, SW9 RotaryEncoder_Switch, U1 XIAO-RP2040-SMD, U2 OLED_I2C

Commit message: Finished the PCB
Parts:
- D1, D2, D3, D4, D5, D6, D7, D8: footprint (none) -> Diode_THT:D_DO-35_SOD27_P7.62mm_Horizontal
- D9: footprint LED_SMD:LED_WS2812_PLCC6_5.0x5.0mm_P1.6mm -> Connector_JST:JST_XH_B3B-XH-A_1x03_P2.50mm_Vertical
- SW1, SW2, SW3, SW4, SW5, SW6, SW7, SW8: footprint (none) -> My_Footprint:SW_Cherry_MX_1.00u_PCB_Wtih_3D
- SW9: footprint (none) -> Rotary_Encoder:RotaryEncoder_Alps_EC11E-Switch_Vertical_H20mm
- U1: footprint Seeed Studio XIAO Series Library:XIAO-RP2350-DIP -> Seeed Studio XIAO Series Library:XIAO-RP2040-DIP
- U2: footprint Display:ER_OLEDM0.91_1x-I2C -> Display-extra:Display_128x64_096_I2C
Connections:
- net +5V: now also U1.14 (VBUS)
- net A_Encoder: now also U1.11 (D10); no longer U1.10 (D9)
- net B_Encoder: now also U1.10 (D9); no longer U1.11 (D10)
- net COL1: now also U1.4 (D3); no longer U1.1 (D0)
- net COL2: now also U1.3 (D2); no longer U1.2 (D1)
- net COL3: now also U1.2 (D1); no longer U1.3 (D2)
- net COL4: now also U1.1 (D0); no longer U1.4 (D3)
- net GND: now also D9.1 (VSS); no longer D9.6 (VSS)
- net SCL_OLED: now also U1.5 (D4); no longer U1.6 (D5)
- net SDA_OLED: now also U1.6 (D5); no longer U1.5 (D4)
Changed lines of the file:
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@@
 	(wire
 		(pts
+			(xy 274.32 87.63) (xy 266.7 87.63)
+		)
+		(stroke
+			(width 0)
+			(type default)
+		)
+	)
+	(wire
+		(pts
 			(xy 111.76 85.09) (xy 137.16 85.09)
 		)
@@
 	(global_label "COL2"
 		(shape input)
-		(at 220.98 91.44 180)
+		(at 220.98 95.25 180)
 		(fields_autoplaced yes)
 		(effects
@@
 		)
 		(property "Intersheetrefs" "${INTERSHEET_REFS}"
-			(at 213.1567 91.44 0)
+			(at 213.1567 95.25 0)
 			(hide yes)
 			(show_name no)
@@
 	(global_label "SCL_OLED"
 		(shape input)
-		(at 222.25 106.68 180)
+		(at 222.25 102.87 180)
 		(fields_autoplaced yes)
 		(effects
@@
 		)
 		(property "Intersheetrefs" "${INTERSHEET_REFS}"
-			(at 210.012 106.68 0)
+			(at 209.9515 102.87 0)
 			(hide yes)
 			(show_name no)
@@
 	(global_label "B_Encoder"
 		(shape input)
-		(at 267.97 99.06 0)
+		(at 267.97 102.87 0)
 		(fields_autoplaced yes)
 		(effects
@@
 		)
 		(property "Intersheetrefs" "${INTERSHEET_REFS}"
-			(at 280.7522 99.06 0)
+			(at 280.5708 102.87 0)
 			(hide yes)
 			(show_name no)
@@
 	(global_label "COL3"
 		(shape input)
-		(at 220.98 95.25 180)
+		(at 220.98 91.44 180)
 		(fields_autoplaced yes)
 		(effects
@@
 		)
 		(property "Intersheetrefs" "${INTERSHEET_REFS}"
-			(at 213.1567 95.25 0)
+			(at 213.1567 91.44 0)
 			(hide yes)
 			(show_name no)
@@
 	(global_label "SDA_OLED"
 		(shape input)
-		(at 222.25 102.87 180)
+		(at 222.25 106.68 180)
 		(fields_autoplaced yes)
 		(effects
@@
 		)
 		(property "Intersheetrefs" "${INTERSHEET_REFS}"
-			(at 209.9515 102.87 0)
+			(at 210.012 106.68 0)
 			(hide yes)
 			(show_name no)
@@
 	(global_label "A_Encoder"
 		(shape input)
-		(at 267.97 102.87 0)
+		(at 267.97 99.06 0)
 		(fields_autoplaced yes)
 		(effects
@@
 		)
 		(property "Intersheetrefs" "${INTERSHEET_REFS}"
-			(at 280.5708 102.87 0)
+			(at 280.7522 99.06 0)
 			(hide yes)
 			(show_name no)
@@
 	(global_label "COL1"
 		(shape input)
-		(at 220.98 87.63 180)
+		(at 220.98 99.06 180)
 		(fields_autoplaced yes)
 		(effects
@@
 		)
 		(property "Intersheetrefs" "${INTERSHEET_REFS}"
-			(at 213.1567 87.63 0)
+			(at 213.1567 99.06 0)
 			(hide yes)
 			(show_name no)
@@
 	(global_label "COL4"
 		(shape input)
-		(at 220.98 99.06 180)
+		(at 220.98 87.63 180)
 		(fields_autoplaced yes)
 		(effects
@@
 		)
 		(property "Intersheetrefs" "${INTERSHEET_REFS}"
-			(at 213.1567 99.06 0)
+			(at 213.1567 87.63 0)
 			(hide yes)
 			(show_name no)
@@
 			)
 		)
-		(property "Footprint" ""
+		(property "Footprint" "Diode_THT:D_DO-35_SOD27_P7.62mm_Horizontal"
 			(at 162.56 101.6 0)
 			(hide yes)
@@
 			)
 		)
-		(property "Footprint" ""
+		(property "Footprint" "Diode_THT:D_DO-35_SOD27_P7.62mm_Horizontal"
 			(at 137.16 81.28 0)
 			(hide yes)
@@
 			)
 		)
-		(property "Footprint" ""
+		(property "Footprint" "My_Footprint:SW_Cherry_MX_1.00u_PCB_Wtih_3D"
 			(at 114.3 93.98 0)
 			(hide yes)
@@
 			)
 		)
-		(property "Footprint" ""
+		(property "Footprint" "My_Footprint:SW_Cherry_MX_1.00u_PCB_Wtih_3D"
 			(at 139.7 93.98 0)
 			(hide yes)
@@
 			)
 		)
-		(property "Footprint" "Seeed Studio XIAO Series Library:XIAO-RP2350-DIP"
+		(property "Footprint" "Seeed Studio XIAO Series Library:XIAO-RP2040-DIP"
 			(at 249.428 118.872 0)
 			(hide yes)
@@
 			)
 		)
-		(property "Footprint" ""
+		(property "Footprint" "Diode_THT:D_DO-35_SOD27_P7.62mm_Horizontal"
 			(at 162.56 81.28 0)
 			(hide yes)
@@
 			)
 		)
-		(property "Footprint" ""
+		(property "Footprint" "My_Footprint:SW_Cherry_MX_1.00u_PCB_Wtih_3D"
 			(at 165.1 73.66 0)
 			(hide yes)
@@
 			)
 		)
-		(property "Footprint" ""
+		(property "Footprint" "Diode_THT:D_DO-35_SOD27_P7.62mm_Horizontal"
 			(at 111.76 101.6 0)
 			(hide yes)
@@
 			)
 		)
-		(property "Footprint" ""
+		(property "Footprint" "My_Footprint:SW_Cherry_MX_1.00u_PCB_Wtih_3D"
 			(at 190.5 93.98 0)
 			(hide yes)
@@
 			)
 		)
-		(property "Footprint" ""
+		(property "Footprint" "My_Footprint:SW_Cherry_MX_1.00u_PCB_Wtih_3D"
 			(at 139.7 73.66 0)
 			(hide yes)
@@
 			)
 		)
-		(property "Footprint" "Display:ER_OLEDM0.91_1x-I2C"
+		(property "Footprint" "Display-extra:Display_128x64_096_I2C"
 			(at 58.674 100.33 0)
 			(hide yes)
@@
 			)
 		)
-		(property "Footprint" ""
+		(property "Footprint" "My_Footprint:SW_Cherry_MX_1.00u_PCB_Wtih_3D"
 			(at 190.5 73.66 0)
 			(hide yes)
@@
 			)
 		)
-		(property "Footprint" ""
+		(property "Footprint" "Diode_THT:D_DO-35_SOD27_P7.62mm_Horizontal"
 			(at 137.16 101.6 0)
 			(hide yes)
@@
 			)
 		)
-		(property "Footprint" ""
+		(property "Footprint" "Diode_THT:D_DO-35_SOD27_P7.62mm_Horizontal"
 			(at 111.76 81.28 0)
 			(hide yes)
@@
 			)
 		)
-		(property "Footprint" ""
+		(property "Footprint" "Diode_THT:D_DO-35_SOD27_P7.62mm_Horizontal"
 			(at 187.96 81.28 0)
 			(hide yes)
@@
 			)
 		)
-		(property "Footprint" ""
+		(property "Footprint" "Rotary_Encoder:RotaryEncoder_Alps_EC11E-Switch_Vertical_H20mm"
 			(at 57.15 111.506 0)
 			(hide yes)
@@
 	)
 	(symbol
+		(lib_id "power:+5V")
+		(at 274.32 87.63 0)
+		(unit 1)
+		(body_style 1)
+		(exclude_from_sim no)
+		(in_bom yes)
+		(on_board yes)
+		(in_pos_files yes)
+		(dnp no)
+		(fields_autoplaced yes)
+		(property "Reference" "#PWR010"
+			(at 274.32 91.44 0)
+			(hide yes)
+			(show_name no)
+			(do_not_autoplace no)
+			(effects
+				(font
+					(size 1.27 1.27)
+				)
+			)
+		)
+		(property "Value" "+5V"
+			(at 274.32 82.55 0)
+			(show_name no)
+			(do_not_autoplace no)
+			(effects
+				(font
+					(size 1.27 1.27)
+				)
+			)
+		)
+		(property "Footprint" ""
+			(at 274.32 87.63 0)
+			(hide yes)
+			(show_name no)
+			(do_not_autoplace no)
+			(effects
+				(font
+					(size 1.27 1.27)
+				)
+			)
+		)
+		(property "Datasheet" ""
+			(at 274.32 87.63 0)
+			(hide yes)
+			(show_name no)
+			(do_not_autoplace no)
+			(effects
+				(font
+					(size 1.27 1.27)
+				)
+			)
+		)
+		(property "Description" "Power symbol creates a global label with name \"+5V\""
+			(at 274.32 87.63 0)
+			(hide yes)
+			(show_name no)
+			(do_not_autoplace no)
+			(effects
+				(font
+					(size 1.27 1.27)
+				)
+			)
+		)
+		(pin "1"
+		)
+		(instances
+			(project "BoxPad_PCB"
+				(path "/eb0de2ab-bbc4-4aaa-ab20-7cc73d5ad5e7"
+					(reference "#PWR010")
+					(unit 1)
+				)
+			)
+		)
+	)
+	(symbol
 		(lib_id "power:GND")
 		(at 35.56 115.57 0)
@@
 			)
 		)
-		(property "Footprint" "LED_SMD:LED_WS2812_PLCC6_5.0x5.0mm_P1.6mm"
+		(property "Footprint" "Connector_JST:JST_XH_B3B-XH-A_1x03_P2.50mm_Vertical"
 			(at 78.74 96.52 0)
 			(hide yes)
@@
 		)
 		(property "Description" "RGB LED with integrated controller"
-			(at 77.47 88.9 0)
+			(at 99.06 78.994 0)
 			(hide yes)
 			(show_name no)
@@
 			)
 		)
-		(property "Footprint" ""
+		(property "Footprint" "My_Footprint:SW_Cherry_MX_1.00u_PCB_Wtih_3D"
 			(at 114.3 73.66 0)
 			(hide yes)
@@
 			)
 		)
-		(property "Footprint" ""
+		(property "Footprint" "My_Footprint:SW_Cherry_MX_1.00u_PCB_Wtih_3D"
 			(at 165.1 93.98 0)
 			(hide yes)
@@
 			)
 		)
-		(property "Footprint" ""
+		(property "Footprint" "Diode_THT:D_DO-35_SOD27_P7.62mm_Horizontal"
 			(at 187.96 101.6 0)
 			(hide yes)
